File: miniSpartan6+_Rev_B.sch (EAGLE design)
At the start: 95 parts, among them J1 USB-MINIB-5PIN, J2 HDMI-TYPE-A-RECEPTICALFCI1002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, J3 HDMI-TYPE-A-RECEPTICALFCI1002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, J4 P24-1, J5 MICROSD_MOLEX, J6 P24-1, Q1 12MHz, U1 93C46B, U10 SPI_FLASH-SOIC_150_208, U11 PCA9306, U3 ADC088S102CIMT, U4 +3.3V Reg., U5 +1.2V Reg., U6 XC6SLX25-FT256, U7 ASFLMB-32.000MHZ-LC-T, U8 ASFLMB-50.000MHZ-LC-T, U9 SDRAM-16MX16-WINBOND

Commit message: Updating to the current production version
Parts:
- removed J1: USB-MINIB-5PIN, saanlima:USB-MINIB-5PIN
- added C37, C39, C40: .1uF, rcl:C-EUC0603K
- added R7: 0, rcl:R-US_R0603
- added RN8, RN9: 51, resistor-dil:2R-NEXB34V
- added X1: MINI-USB-UX60-MB-5S8, con-hirose:MINI-USB-UX60-MB-5S8
- C11, C13: value (none) -> 4.7uF
- R4: value 0DNI -> 470
- R5: value 0 -> 470
- RN1, RN2: value (none) -> 1k
- RN3, RN4: value (none) -> 51; device resistor-dil:4R-N0603-ARV -> resistor-dil:2R-NEXB34V
- RN5: value (none) -> 2k
- U2: value (none) -> FT2232HL
Connections:
- net IO0 renamed PORTA0
- net IO1 renamed PORTA1
- net IO11 renamed PORTA11
- net IO12 renamed PORTB0
- net IO13 renamed PORTB1
- net IO14 renamed PORTB2
- net IO15 renamed PORTB3
- net IO16 renamed PORTB4
- net IO17 renamed PORTB5
- net IO18 renamed PORTB6
- net IO19 renamed PORTB7
- net IO2 renamed PORTA2
- net IO20 renamed PORTB8
- net IO21 renamed PORTB9
- net IO22 renamed PORTB10
- net IO23 renamed PORTB11
- net IO24 renamed PORTC0
- net IO25 renamed PORTC1
- net IO26 renamed PORTC2
- net IO27 renamed PORTC3
- net IO28 renamed PORTC4
- net IO29 renamed PORTC5
- net IO3 renamed PORTA3
- net IO30 renamed PORTC6
- net IO31 renamed PORTC7
- net IO32 renamed PORTC8
- net IO33 renamed PORTC9
- net IO34 renamed PORTC10
- net IO35 renamed PORTC11
- net IO36 renamed PORTD0
- net IO37 renamed PORTD1
- net IO38 renamed PORTD2
- net IO39 renamed PORTD3
- net IO42 renamed PORTE2
- net IO43 renamed PORTE3
- net IO48 renamed PORTE8
- net IO49 renamed PORTE9
- net IO5 renamed PORTA5
- net IO50 renamed PORTE10
- net IO51 renamed PORTE11
- net IO54 renamed PORTF2
- net IO55 renamed PORTF3
- net IO56 renamed PORTF4
- net IO57 renamed PORTF5
- net IO6 renamed PORTA6
- net IO60 renamed PORTF8
- net IO61 renamed PORTF9
- net IO62 renamed PORTF10
- net IO63 renamed PORTF11
- removed net CEC: J3.CEC
- removed net IO10: U$7.P7, U6IO_L37P_GCLK13_0.1
- removed net IO4: U$7.P3, U6IO_L34N_GCLK18_0.1
- removed net IO40: J4.P9, U6IO_L3P_0.1
- removed net IO41: J6.P9, U6IO_L1N_VREF_0.1
- removed net IO44: J4.P12, U6IO_L52N_M3A9_3.1
- removed net IO45: J6.P12, U6IO_L83P_3.1
- removed net IO46: J4.P13, U6IO_L52P_M3A8_3.1
- removed net IO47: J6.P13, U6IO_L48P_M3BA0_3.1
- removed net IO52: J4.P17, U6IO_L46P_M3CLK_3.1
- removed net IO53: J6.P17, U6IO_L46N_M3CLKN_3.1
- removed net IO58: J4.P21, U6IO_L53N_M3A12_3.1
- removed net IO59: J6.P21, U6IO_L40N_M3DQ7_3.1
- removed net IO7: U$8.P5, U6IO_L34P_GCLK19_0.1
- removed net IO8: U$7.P6, U6IO_L37N_GCLK12_0.1
- removed net IO9: U$8.P6, U6IO_L40N_0.1
- removed net N$22: J1.MTN1, J1.MTN2, R1.2
- removed net N$35: R5.2, RN3A.1, RN3B.1, RN3C.1, RN3D.1, RN4A.1, RN4B.1, RN4C.1, RN4D.1
- new net N$13: C37.1, R1.2, X1.M1, X1.M2, X1.M3, X1.M4
- new net N$8: R7.2, RN3A.1, RN3B.2, RN4A.1, RN4B.2, RN8A.1, RN8B.2, RN9A.1, RN9B.2
- new net PORTA10: U$7.P7, U6IO_L64P_SCP5_0.1
- new net PORTA4: U$7.P3, U6IO_L40N_0.1
- new net PORTA7: U$8.P5, U6IO_L37N_GCLK12_0.1
- new net PORTA8: U$7.P6, U6IO_L37P_GCLK13_0.1
- new net PORTA9: U$8.P6, U6IO_L40P_0.1
- new net PORTE0: J4.P10, U6IO_L3P_0.1
- new net PORTE1: J6.P10, U6IO_L1N_VREF_0.1
- new net PORTE4: J4.P12, U6IO_L83P_3.1
- new net PORTE5: J6.P12, U6IO_L52N_M3A9_3.1
- new net PORTE6: J4.P14, U6IO_L52P_M3A8_3.1
- new net PORTE7: J6.P14, U6IO_L48P_M3BA0_3.1
- new net PORTF0: J4.P18, U6IO_L46P_M3CLK_3.1
- new net PORTF1: J6.P18, U6IO_L46N_M3CLKN_3.1
- new net PORTF6: J4.P22, U6IO_L53N_M3A12_3.1
- new net PORTF7: J6.P22, U6IO_L40N_M3DQ7_3.1
- net 1V2: now also R5.2
- net 3V3: now also J4.P13, J4.P21, J6.P17, J6.P9, R4.2, R7.1; no longer J4.P14, J4.P22, J6.P10, J6.P18, R5.1
- net 5V0: now also X1.1; no longer J1.VBUS, R4.2
- net AD_DIN: now also U6IO_L44P_GCLK21_M3A5_3.1; no longer U6IO_L51P_M3A10_3.1
- net AD_SCLK: now also U6IO_L51P_M3A10_3.1; no longer U6IO_L44P_GCLK21_M3A5_3.1
- net AUDIO1: now also U6IO_L33P_0.1; no longer U6IO_L50N_M3BA2_3.1
- net AUDIO2: now also U6IO_L33N_0.1; no longer U6IO_L50P_M3WE_3.1
- net A_TMDS0_N: no longer RN4B.2
- net A_TMDS0_P: no longer RN4A.2
- net A_TMDS1_N: no longer RN3D.2
- net A_TMDS1_P: no longer RN3C.2
- net A_TMDS2_N: no longer RN3B.2
- net A_TMDS2_P: no longer RN3A.2
- net A_TMDS_CLK_N: no longer RN4D.2
- net A_TMDS_CLK_P: no longer RN4C.2
- net DDC_SCL: now also J2.SCL; no longer J3.SCL
- net DDC_SDA: now also J2.SDA; no longer J3.SDA
- net FPGA-CLK-2: now also U6IO_L42N_GCLK24_M3LDM_3.1; no longer U6IO_L41N_GCLK26_M3DQ5_3.1
- net FPGA_SCL: now also U6IO_L50P_M3WE_3.1
- net FPGA_SDA: now also U6IO_L50N_M3BA2_3.1
- net GND: now also C37.2, C39.2, C40.2, J4.P17, J4.P9, J6.P13, J6.P21, R4.1, R5.1, X1.5; no longer J1.GND, J4.P10, J4.P18, J6.P14, J6.P22, R14.1
- net N$10: now also X1.2; no longer J1.D-
- net N$14: now also X1.3; no longer J1.D+
- net N$24: now also JP5.TIP; no longer JP5.RING1
- net N$25: now also JP5.RING1; no longer JP5.TIP
- net N$34: now also C39.1
- net N$36: now also C40.1
- net TMDS0_N: now also RN8A.2
- net TMDS0_P: now also RN8B.1
- net TMDS1_N: now also RN3A.2
- net TMDS1_P: now also RN3B.1
- net TMDS2_N: now also RN4A.2
- net TMDS2_P: now also RN4B.1
- net TMDS_CLK_N: now also RN9A.2, U6IO_L34N_GCLK18_0.1; no longer U6IO_L33N_0.1
- net TMDS_CLK_P: now also RN9B.1, U6IO_L34P_GCLK19_0.1; no longer U6IO_L33P_0.1
- net TX_HDMI_5V: now also J2.+5V, R14.1; no longer J3.+5V, R4.1
Other:
- moved on the sheet: C11, C13, C33, J2, L3, R14, R19, R2, R20, R3, R6, RN3A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

Commit message: Added Copyright to the schematic
Added Copyright to the schematic
Other:
- note added: "Copyright Scarab Hardware 2014 With some parts from Saanlima Electronics Under Creative Commons Attribution Sharealike 4.0"
- moved on the sheet: C16, C17, C18, C19, C20, C21, C22, C23, C24, C25, C26, C27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
